File: Hardware/sparkfun-samd21g18-r3.brd (EAGLE design)
At the start: 57.1 x 53.3 mm, 59 parts, among them Q1 2.5A/30V, Q2 2N7002PW, U1 MCP73831, U2 74AHC1G125, U3 MIC5219 3.3V, U4 ATSAMD21G-A

Commit message: Minor fixes for pre-QC check.
Parts:
- C7, C9: value 22pF -> 15pF
- D5: value Yellow -> GREEN
- D6: value GREEN -> Yellow
- JP1: device SparkFun-Connectors:USB-AB-MICRO-SMD_V03 -> SparkFun-Connectors:1X02
- JP2: device SparkFun-Connectors:1X02 -> SparkFun-Connectors:USB-AB-MICRO-SMD_V03
- LOGO2: value OSHW-LOGOS -> SFE_LOGO_NAME_FLAME.4_INCH; device SparkFun-Aesthetics:OSHW-LOGO-S -> SparkFun-Aesthetics:SFE_LOGO_NAME_FLAME_.4
- LOGO3: value SFE_LOGO_NAME_FLAME.4_INCH -> OSHW-LOGOS; device SparkFun-Aesthetics:SFE_LOGO_NAME_FLAME_.4 -> SparkFun-Aesthetics:OSHW-LOGO-S
- Y1: value (none) -> 32.768kHz
- moved STANDOFF2 66.7 mm to (3.81, 50.8)
- moved LOGO2 60.5 mm to (50.8, 7.62), flipped to the bottom, turned to 45 degrees
- moved LOGO3 60.5 mm to (3.81, 45.7), flipped to the top, turned to 0 degrees
- moved STANDOFF1 52.3 mm to (54.6, 7.62)
- moved STANDOFF3 48.3 mm to (2.54, 2.54)
- moved JP1 29.2 mm to (1.27, 8.89), turned to 90 degrees
- moved JP2 29.2 mm to (2.29, 38.1), turned to 0 degrees
- renumbered JP8 to JP5
Connections:
- net N$14 renamed CHG_STAT
- removed net 5V: C3.1, C4.1, D1.C, D2.A, JP2.2, JP3.PWR, JP7.VIN, Q1.2, R5.2, U1.4, U3.1, U3.3
- new net VIN: C3.1, C4.1, D1.C, D2.A, JP1.2, JP3.PWR, JP7.VIN, Q1.2, R5.2, U1.4, U3.1, U3.3
- net GND: now also JP1.1, JP2.GND1, JP2.SHIELD1, JP2.SHIELD2, JP2.SHIELD3; no longer JP1.GND1, JP1.SHIELD1, JP1.SHIELD2, JP1.SHIELD3, JP2.1
- net N$1: now also JP2.VBUS1; no longer JP1.VBUS1
- net USB_D+: now also JP2.D+1; no longer JP1.D+1
- net USB_D-: now also JP2.D-1; no longer JP1.D-1
- net USB_ID: now also JP2.ID1; no longer JP1.ID1
Routing:
- net VIN: track 0.00 -> 119.1 mm, vias 0 -> 2
- net 5V: track 119.1 -> 0.00 mm, vias 2 -> 0
- net A5: track 34.0 -> 31.0 mm
Other:
- board text added: "Jim Lindblom"
- board text removed: "SAMD21 R3 Breakout"

Commit message: Adding SMD JST package, moving LEDs and USB to accomodate.
Parts:
- added JP8: (no value), SparkFun-Connectors:JST-2-PTH-NS
- JP4: device SparkFun-Connectors:JST-2-PTH -> SparkFun-Connectors:JST-2-SMD
- moved D2 3.18 mm to (2.54, 24.8)
- moved D6 3.18 mm to (2.54, 27.3)
- moved R10 3.18 mm to (2.54, 26.0)
- moved R7 3.18 mm to (2.54, 33.7)
- moved R9 3.18 mm to (2.54, 28.6)
- moved D3 3.17 mm to (2.54, 34.9)
- moved D4 3.17 mm to (2.54, 32.4)
- moved D5 3.17 mm to (2.54, 29.8)
- moved Q2 3.17 mm to (7.62, 32.4)
- moved R8 3.17 mm to (2.54, 31.1)
- moved SJ2 3.17 mm to (5.08, 34.9)
- moved JP4 2.84 mm to (3.56, 19.2)
- moved D1 2.84 mm to (12.7, 19.1), turned to 90 degrees
- moved JP2 2.54 mm to (2.29, 40.6)
- moved C1 1.27 mm to (10.2, 43.2)
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Connections:
- net GND: now also JP8.1
- net VBAT: now also JP8.2
Routing:
- net VIN: track 119.1 -> 131.5 mm, vias 2 -> 3
- net VUSB: track 76.1 -> 79.4 mm
- net USB_HOST_POWER_EN: track 33.6 -> 35.7 mm
- net VBAT: track 14.4 -> 12.4 mm
- net GND: track 30.5 -> 32.3 mm, vias 16 -> 15
- net D13: track 62.6 -> 64.0 mm
- net TX_LED: track 37.6 -> 38.9 mm
- net USB_D-: track 32.8 -> 33.9 mm
- net USB_D+: track 32.7 -> 33.8 mm
- net USB_ID: track 16.3 -> 17.3 mm
- net N$8: track 7.16 -> 7.95 mm
- net N$1: track 3.46 -> 2.70 mm
- net CHG_STAT: track 8.29 -> 7.77 mm
