File: Hardware/sparkfun-samd21g18-r3.sch (EAGLE design)
At the start: 59 parts, among them Q1 2.5A/30V, Q2 2N7002PW, U1 MCP73831, U2 74AHC1G125, U3 MIC5219 3.3V, U4 ATSAMD21G-A

Commit message: Minor fixes for pre-QC check.
Parts:
- C7, C9: value 22pF -> 15pF; device SparkFun-Capacitors:22PF-50V-5%(0603) -> SparkFun-Capacitors:15PF-50V-5%(0603)
- D5: value Yellow -> GREEN; device SparkFun-LED:LED-YELLOW0603 -> SparkFun-LED:LED-GREEN0603
- D6: value GREEN -> Yellow; device SparkFun-LED:LED-GREEN0603 -> SparkFun-LED:LED-YELLOW0603
- JP1: device SparkFun-Connectors:USB-ABCONN-11794 -> SparkFun-Connectors:M02PTH
- JP2: device SparkFun-Connectors:M02PTH -> SparkFun-Connectors:USB-ABCONN-11794
- LOGO2: value OSHW-LOGOS -> SFE_LOGO_NAME_FLAME.4_INCH; device SparkFun-Aesthetics:OSHW-LOGOS -> SparkFun-Aesthetics:SFE_LOGO_NAME_FLAME.4_INCH
- LOGO3: value SFE_LOGO_NAME_FLAME.4_INCH -> OSHW-LOGOS; device SparkFun-Aesthetics:SFE_LOGO_NAME_FLAME.4_INCH -> SparkFun-Aesthetics:OSHW-LOGOS
- Y1: value (none) -> 32.768kHz
- renumbered JP8 to JP5
Connections:
- net N$14 renamed CHG_STAT
- removed net 5V: C3.1, C4.1, D1.C, D2.A, JP2.2, JP3.PWR, JP7.VIN, Q1.S, R5.2, U1.VIN, U3.EN, U3.IN
- new net VIN: C3.1, C4.1, D1.C, D2.A, JP1.2, JP3.PWR, JP7.VIN, Q1.S, R5.2, U1.VIN, U3.EN, U3.IN
- net GND: now also JP1.1, JP2.GND, JP2.SHIELD; no longer JP1.GND, JP1.SHIELD, JP2.1
- net N$1: now also JP2.VBUS; no longer JP1.VBUS
- net USB_D+: now also JP2.D+; no longer JP1.D+
- net USB_D-: now also JP2.D-; no longer JP1.D-
- net USB_ID: now also JP2.USBID; no longer JP1.USBID
Other:
- note added: "ATSAMD21G18 VDD Range: 1.62-3.63V"
- note added: "VIN must be 4.5-5.5V, if battery charger is used"
- moved on the sheet: D2, D3, R6, R7, SJ2

Commit message: Adding SMD JST package, moving LEDs and USB to accomodate.
Parts:
- added JP8: (no value), SparkFun-Connectors:M02-JST-2-PTH-NO_SILK
- JP4: device SparkFun-Connectors:M02JST-PTH-2 -> SparkFun-Connectors:M02-JST-2MM-SMT
Connections:
- net GND: now also JP4.2, JP8.1; no longer JP4.1
- net VBAT: now also JP4.1, JP8.2; no longer JP4.2
Other:
- moved on the sheet: JP4
