File: Hardware/sparkfun-samd21g-r3.sch (EAGLE design)
At the start: 62 parts, among them Q1 2.5A/30V, Q2 2N7002PW, U1 MCP73831, U2 74AHC1G125, U3 3.3V, U4 ATSAMD21G-A, Y1 32.768kHz

Commit message: Tweaking schematic and layout silk for checklist
Other:
- note added: "0.1" Header"
- note added: "2-Pin PTH JST"
- note added: "2-pin SMD JST"
- note added: "AP2112K-3.3V ---------------- Iout (max): 600mA Vin (max): 6.5V Vdrop (max): 250mV Iq: 55uA"
- note added: "Based on: Arduino Zero by Arduino.cc Arduino M0 by Arduino.org"
- note added: "Pins routed to the EDBG or SWD. Equivalent Arduino pin labeled on board"
- note added: "USB Host/Device Control ----------------------------- - USB_ID High: Y high, Q1 off - USB_ID Low: Y low, Q1 on - Set USB_HOST_EN low to turn Q1 on and route power OUT the board. - USB_HOST_EN floating or HIGH turns Q1 off. USB supply flows through Q1 body diode."
- note added: "VBAT: 3.6-4.2V Single cell LiPo battery only\!"
- note removed: "USB Host/Device Control"
- moved on the sheet: C10, C2, C4, C6, C7, C9, D1, JP4, JP5, JP7, JP8, JP9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

Commit message: Fixing typo in comment about SJ1.
Other:
- note added: "SJ1 connects/disconnects R1 from the MCP73831 PROG input. Cut the jumper if you want to use a custom resistor value."
- note removed: "SJ1 connects/disconnects R9 from the MCP73831 PROG input. Cut the jumper if you want to use a custom resistor value."
Changed lines of the file:
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@@
 <text x="43.18" y="40.64" size="1.778" layer="97" rot="R180">Charge Current=
 ~256mA (1000V/3900)</text>
-<text x="50.8" y="50.8" size="1.778" layer="97" align="bottom-right">SJ1 connects/disconnects R9
+<text x="50.8" y="50.8" size="1.778" layer="97" align="bottom-right">SJ1 connects/disconnects R1
 from the MCP73831 PROG input.
 Cut the jumper if you want to
